Commit message: Changes

File: uuv_sensor_plugins/uuv_sensor_ros_plugins/urdf/camera_snippets.xacro (robot description, xacro)
@@ -23,5 +23,5 @@
   </xacro:macro>
   <xacro:macro name="default_camera" params="namespace parent_link suffix *origin">
-    <xacro:regular_camera_plugin_macro
+    <xacro:underwater_camera_plugin_macro
       namespace="${namespace}"
       suffix="${suffix}"
@@ -34,8 +34,11 @@
       height="492"
       stddev="0.02"
-      scale="1.0">
+      scale="1.0"
+      offset_x="0.049"
+      offset_y="0"
+      offset_z="0.053">
       <inertia ixx="0.00001" ixy="0.0" ixz="0.0" iyy="0.00001" iyz="0.0" izz="0.00001" />
       <xacro:insert_block name="origin" />
-    </xacro:regular_camera_plugin_macro>
+    </xacro:underwater_camera_plugin_macro>
   </xacro:macro>
   <xacro:macro name="wideangle_camera" params="namespace parent_link suffix *origin">
@@ -69,5 +72,5 @@
       <visual>
         <geometry>
-          <mesh filename="file://$(find uuv_sensor_ros_plugins)/meshes/oe14-372.dae" scale="${scale} ${scale} ${scale}"/>
+          <mesh filename="file://$(find uuv_sensor_ros_plugins)/meshes/zedmini_camera.dae" scale="${scale} ${scale} ${scale}"/>
         </geometry>
       </visual>
@@ -141,88 +144,182 @@
     </gazebo>
   </xacro:macro>
-  <xacro:macro name="underwater_camera_plugin_macro"
-    params="namespace suffix parent_link topic mass update_rate
-      hfov width height stddev
+  <xacro:macro name="underwater_camera_plugin_macro" params="offset_x offset_y offset_z namespace suffix parent_link topic mass update_rate
+      hfov width height stddev scale
       *inertia *origin">
-    <!-- Sensor link -->
-    <link name="${namespace}/camera${suffix}_link">
-      <inertial>
-        <xacro:insert_block name="inertia" />
-        <mass value="${mass}" />
-        <origin xyz="0 0 0" rpy="0 0 0" />
-      </inertial>
-      <visual>
-        <geometry>
-          <mesh filename="file://$(find uuv_sensor_ros_plugins)/meshes/oe14-372.dae" scale="1 1 1"/>
-        </geometry>
-      </visual>
-      <xacro:no_collision/>
+    <!-- Camera link -->
+    <link name="${suffix}rs200_camera">
+        <visual>
+            <origin rpy="0 0 0" xyz="0 0 0"/>
+            <geometry>
+                <mesh filename="package://realsense_gazebo_plugin/models/realsense_camera/meshes/realsense.dae"/>
+            </geometry>
+        </visual>
+        <collision>
+            <geometry>
+                <box size="0.0078 0.130 0.0192"/>
+            </geometry>
+        </collision>
+        <inertial>
+            <mass value="0.0615752"/>
+            <origin rpy="0 0 0" xyz="0 0 0"/>
+            <inertia ixx="9.108e-05"
+                     ixy="0"
+                     ixz="0"
+                     iyy="2.51e-06"
+                     iyz="0"
+                     izz="8.931e-05"
+            />
+        </inertial>
     </link>
-    <joint name="${namespace}/camera${suffix}_joint" type="revolute">
-      <xacro:insert_block name="origin" />
-      <parent link="${parent_link}" />
-      <child link="${namespace}/camera${suffix}_link" />
-      <axis xyz="1 0 0"/>
-      <limit upper="0" lower="0" effort="0" velocity="0" />
-    </joint>
-    <link name="${namespace}/camera${suffix}_link_optical">
-      <xacro:box_inertial x="0.0001" y="0.0001" z="0.0001" mass="0.001">
-        <origin xyz="0 0 0" rpy="0 0 0"/>
-      </xacro:box_inertial>
-      <collision>
-        <!-- todo: gazebo needs a collision volume or it will ignore the pose of
-           the joint that leads to this link (and assume it to be the identity) -->
-        <geometry>
-          <cylinder length="0.000001" radius="0.000001"/>
-        </geometry>
-        <origin xyz="0 0 0" rpy="0 ${0.5*pi} 0"/>
-      </collision>
-    </link>
-    <joint name="${namespace}/camera${suffix}_optical_joint" type="revolute">
-      <origin xyz="0 0 0" rpy="${-pi/2} 0 ${-pi/2}"/>
-      <parent link="${namespace}/camera${suffix}_link"/>
-      <child link="${namespace}/camera${suffix}_link_optical"/>
-      <limit upper="0" lower="0" effort="0" velocity="0" />
-      <axis xyz="1 0 0"/>
-    </joint>
-    <gazebo reference="${namespace}/camera${suffix}_link">
-      <sensor type="depth" name="camera${suffix}">
-        <update_rate>${update_rate}</update_rate>
-        <camera name="camera${suffix}">
-          <horizontal_fov>${hfov}</horizontal_fov>
-          <image>
-            <width>${width}</width>
-            <height>${height}</height>
-            <format>R8G8B8</format>
-          </image>
-          <clip>
-            <near>0.1</near>
-            <far>3000</far>
-          </clip>
-          <noise>
-            <type>gaussian</type>
-            <mean>0.0</mean>
-            <stddev>${stddev}</stddev>
-          </noise>
-        </camera>
-        <plugin name="camera${suffix}_controller" filename="libuuv_gazebo_ros_camera_plugin.so">
-          <updateRate>${update_rate}</updateRate>
-          <cameraName>${namespace}/camera${suffix}</cameraName>
-          <frameName>${namespace}/camera${suffix}_link</frameName>
-          <attenuationR>0.01</attenuationR>
-          <attenuationG>0.01</attenuationG>
-          <attenuationB>0.003</attenuationB>
-          <backgroundR>0</backgroundR>
-          <backgroundG>0</backgroundG>
-          <backgroundB>0</backgroundB>
-          <!-- required for ros depth cam -->
-          <imageTopicName>${topic}_image</imageTopicName>
-          <pointCloudTopicName>${topic}_cloud</pointCloudTopicName>
-          <depthImageTopicName>${topic}_depth</depthImageTopicName>
-          <depthImageCameraInfoTopicName>${topic}_depth_info</depthImageCameraInfoTopicName>
-          <pointCloudCutoff>10.0</pointCloudCutoff>
+    <!-- Connect camera to parent frame-->
+    <joint name="${suffix}realsense_joint" type="fixed">
+        <parent link="${parent_link}"/>
+        <child link="${suffix}rs200_camera"/>
+        <xacro:insert_block name="origin"/>
+    </joint>
+    <!-- Virtual links representing the cameras positons and orientations-->
+    <link name="${suffix}color" />
+    <link name="${suffix}depth" />
+    <link name="${suffix}ired1" />
+    <link name="${suffix}ired2" />
+    <!-- Joints positioning the virtual links with respect to the camera main link-->
+    <joint name="${suffix}color_joint" type="fixed">
+        <parent link="${suffix}rs200_camera" />
+        <child link="${suffix}color" />
+        <!-- <origin xyz="0 -0.046 0.004" rpy="0 0 0"/> -->
+        <!-- The default position is change since in Rviz the cloud depth axis is Z not X-->
+        <origin xyz="0 -0.046 0.004" rpy="${pi/2} ${pi} ${pi/2}"/>
+    </joint>
+    <joint name="${suffix}depth_joint" type="fixed">
+        <parent link="${suffix}rs200_camera" />
+        <child link="${suffix}depth" />
+        <origin xyz="0 -0.03 0.004" rpy="0 0 0"/>
+    </joint>
+    <joint name="${suffix}ired1_joint" type="fixed">
+        <parent link="${suffix}rs200_camera" />
+        <child link="${suffix}ired1" />
+        <origin xyz="0 -0.06 0.004" rpy="0 0 0"/>
+    </joint>
+    <joint name="${suffix}ired2_joint" type="fixed">
+        <parent link="${suffix}rs200_camera" />
+        <child link="${suffix}ired2" />
+        <origin xyz="0 0.01 0.004" rpy="0 0 0"/>
+    </joint>
+<!-- **********************************************************-->
+<!-- GAZEBO DEFINITIONS ***************************************-->
+    <!-- Load plugin to the model ("robot" in urdf format)-->
+    <gazebo>
+        <plugin name="${suffix}r200" filename="librealsense_gazebo_plugin.so">
+            <prefix>${suffix}</prefix>
         </plugin>
-      </sensor>
+        <!--<pose frame="">0 0 0.015 0 0 0</pose>-->
     </gazebo>
+    <!-- Load parameters to model's main link-->
+    <gazebo reference="${suffix}rs200_camera">
+        <self_collide>0</self_collide>
+        <enable_wind>0</enable_wind>
+        <kinematic>0</kinematic>
+        <gravity>1</gravity>
+        <!--<mu>1</mu>-->
+        <mu2>1</mu2>
+        <fdir1>0 0 0</fdir1>
+        <!--<slip1>0</slip1>
+        <slip2>0</slip2>-->
+        <kp>1e+13</kp>
+        <kd>1</kd>
+        <!--<max_vel>0.01</max_vel>
+        <min_depth>0</min_depth>-->
+        <sensor name="${suffix}color" type="camera">
+            <pose frame="">0 -0.046 0.004 0 0 0</pose>
+            <camera name="${suffix}rs200_camera">
+            <horizontal_fov>1.047</horizontal_fov>
+            <image>
+                <width>640</width>
+                <height>480</height>
+                <format>RGB_INT8</format>
+            </image>
+            <clip>
+                <near>0.1</near>
+                <far>100</far>
+            </clip>
+            <noise>
+                <type>gaussian</type>
+                <mean>0.0</mean>
+                <stddev>0.007</stddev>
+            </noise>
+            </camera>
+            <always_on>1</always_on>
+            <update_rate>60</update_rate>
+            <visualize>1</visualize>
+        </sensor>
+        <sensor name="${suffix}ired1" type="camera">
+            <pose frame="">0 -0.06 0.004 0 0 0</pose>
+            <camera name="${suffix}rs200_camera">
+            <horizontal_fov>1.047</horizontal_fov>
+            <image>
+                <width>640</width>
+                <height>480</height>
+                <format>L_INT8</format>
+            </image>
+            <clip>
+                <near>0.1</near>
+                <far>100</far>
+            </clip>
+            <noise>
+                <type>gaussian</type>
+                <mean>0.0</mean>
+                <stddev>0.05</stddev>
+            </noise>
+            </camera>
+            <always_on>1</always_on>
+            <update_rate>60</update_rate>
+            <visualize>0</visualize>
+        </sensor>
+        <sensor name="${suffix}ired2" type="camera">
+            <pose frame="">0 0.01 0.004 0 0 0</pose>
+            <camera name="${suffix}rs200_camera">
+            <horizontal_fov>1.047</horizontal_fov>
+            <image>
+                <width>640</width>
+                <height>480</height>
+                <format>L_INT8</format>
+            </image>
+            <clip>
+                <near>0.1</near>
+                <far>100</far>
+            </clip>
+            <noise>
+                <type>gaussian</type>
+                <mean>0.0</mean>
+                <stddev>0.05</stddev>
+            </noise>
+            </camera>
+            <always_on>1</always_on>
+            <update_rate>60</update_rate>
+            <visualize>0</visualize>
+        </sensor>
+        <sensor name="${suffix}depth" type="depth">
+            <pose frame="">0 -0.03 0.004 0 0 0</pose>
+            <camera name="${suffix}rs200_camera">
+            <horizontal_fov>1.047</horizontal_fov>
+            <image>
+                    <width>640</width>
+                    <height>480</height>
+            </image>
+            <clip>
+                    <near>0.1</near>
+                    <far>100</far>
+            </clip>
+            <noise>
+                    <type>gaussian</type>
+                    <mean>0.0</mean>
+                    <stddev>0.100</stddev>
+            </noise>
+            </camera>
+            <always_on>1</always_on>
+            <update_rate>60</update_rate>
+            <visualize>0</visualize>
+        </sensor>
+    </gazebo>
   </xacro:macro>
 </robot>

File: uuv_sensor_plugins/uuv_sensor_ros_plugins/urdf/imu_snippets.xacro (robot description, xacro)
@@ -64,5 +64,5 @@
   </xacro:macro>
   <xacro:macro name="default_imu_enu" params="namespace parent_link *origin">
-    <!-- ADIS16448 IMU. -->
+    <!-- ADIS16448 IMU. , have to replace it with Vanttec-IMU-->
     <xacro:imu_plugin_macro
       namespace="${namespace}"
@@ -88,5 +88,5 @@
   </xacro:macro>
   <xacro:macro name="default_imu_ned" params="namespace parent_link *origin">
-    <!-- ADIS16448 IMU. -->
+    <!-- ADIS16448 IMU. have to replace it with Vanttec-IMU-->
     <xacro:imu_plugin_macro
       namespace="${namespace}"

File: uuv_sensor_plugins/uuv_sensor_ros_plugins/urdf/stereo_snippets.xacro (robot description, xacro)
@@ -33,26 +33,64 @@
     </collision>
   </xacro:macro>
-  <xacro:macro name="duo3d_camera" params="namespace parent_link *origin">
-    <link name="${namespace}/duo3d_left_link">
+  <xacro:macro name="stereo_camera" params="namespace parent_link suffix *origin">
+    <link name="duo3d_left_link_stabilized_${suffix}">
+      <inertial>
+        <mass value="0.01"/>
+        <inertia ixx="0.0001" ixy="0" ixz="0" iyy="0.0001" iyz="0" izz="0.0001" />
+      </inertial>
+      <visual>
+        <geometry>
+          <mesh filename="file://$(find uuv_sensor_ros_plugins)/meshes/duo3d.dae"/>
+        </geometry>
+      </visual>
+      <xacro:no_collision/>
+    </link>
+    <joint name="duo3d_stabilized_joint_${suffix}" type="fixed">
+      <xacro:insert_block name="origin" />
+      <preserveFixedJoint>true</preserveFixedJoint>
+      <parent link="${parent_link}"/>
+      <child link="duo3d_left_link_stabilized_${suffix}"/>
+    </joint>
+    <link name="duo3d_left_link_${suffix}">
       <inertial>
         <mass value="0.01"/>
         <inertia ixx="0" ixy="0.0" ixz="0.0" iyy="0" iyz="0.0" izz="0" />
       </inertial>
+      <xacro:no_collision/>
+    </link>
+    <joint name="duo3d_joint_${suffix}" type="fixed">
+      <axis xyz="0 0 1"/>
+      <origin xyz="0 0 0" rpy="0 0 0"/>
+      <parent link="duo3d_left_link_stabilized_${suffix}" />
+      <child link="duo3d_left_link_${suffix}" />
+      <limit upper="0" lower="0" effort="0" velocity="0" />
+    </joint>
+    <joint name="duo3d_optical_joint_${suffix}" type="revolute">
+      <origin xyz="0 0 0" rpy="${-pi/2} 0 ${-pi/2}"/>
+      <parent link="duo3d_left_link_${suffix}"/>
+      <child link="duo3d_optical_link_${suffix}"/>
+      <limit upper="0" lower="0" effort="0" velocity="0" />
+      <axis xyz="1 0 0"/>
+    </joint>
+    <link name="duo3d_optical_link_${suffix}">
+      <xacro:box_inertial x="0.0001" y="0.0001" z="0.0001" mass="0.001">
+        <origin xyz="0 0 0" rpy="0 0 0"/>
+      </xacro:box_inertial>
+      <collision>
+        <!-- todo: gazebo needs a collision volume or it will ignore the pose of
+           the joint that leads to this link (and assume it to be the identity) -->
+        <geometry>
+          <cylinder length="0.000001" radius="0.000001"/>
+        </geometry>
+        <origin xyz="0 0 0" rpy="0 ${0.5*pi} 0"/>
+      </collision>
       <visual>
         <geometry>
-          <mesh filename="file://$(find uuv_sensor_ros_plugins)/meshes/duo3d.dae"/>
+          <cylinder length="0.000001" radius="0.000001"/>
         </geometry>
       </visual>
-      <xacro:no_collision/>
-    </link>
-    <joint name="${namespace}/duo3d_joint" type="revolute">
-      <xacro:insert_block name="origin" />
-      <parent link="${parent_link}" />
-      <child link="${namespace}/duo3d_left_link" />
-      <limit upper="0" lower="0" effort="0" velocity="0" />
-      <axis xyz="1 0 0"/>
-    </joint>
-    <gazebo reference="${namespace}/duo3d_left_link">
-      <sensor name="camera" type="camera">
+    </link>
+    <gazebo reference="duo3d_left_link_${suffix}">
+      <sensor name="camera_${suffix}" type="camera">
       <camera>
         <horizontal_fov>${hfov}</horizontal_fov>
@@ -75,12 +113,12 @@
         </distortion>
       </camera>
-      <plugin name="left_controller" filename="libgazebo_ros_camera.so">
+      <plugin name="left_controller_${suffix}" filename="libgazebo_ros_camera.so">
         <alwaysOn>true</alwaysOn>
         <updateRate>30.0</updateRate>
-        <cameraName>${namespace}/duo3d_left</cameraName>
-        <imageTopicName>image_raw</imageTopicName>
+        <cameraName>stereo_camera_left_${suffix}</cameraName>
+        <imageTopicName>camera_image</imageTopicName>
         <cameraInfoTopicName>camera_info</cameraInfoTopicName>
-        <frameName>${namespace}/duo3d_left_link</frameName>
-        <hackBaseline>0.07</hackBaseline>
+        <frameName>/duo3d_optical_link_${suffix}</frameName>
+        <hackBaseline>0.0</hackBaseline>
         <distortionK1>${k1l}</distortionK1>
         <distortionK2>${k2l}</distortionK2>
@@ -94,5 +132,5 @@
     </sensor>
     </gazebo>
-    <link name="${namespace}/duo3d_right_link">
+    <link name="duo3d_right_link_${suffix}">
       <inertial>
         <mass value="0.01"/>
@@ -101,13 +139,38 @@
       <xacro:no_collision/>
     </link>
-    <joint name="${namespace}/duo3d_right_joint" type="revolute">
-      <origin xyz="0.0 -0.03 0" rpy="0 0 0"/>
-      <parent link="${namespace}/duo3d_left_link" />
-      <child link="${namespace}/duo3d_right_link" />
+    <joint name="duo3d_right_joint_${suffix}" type="fixed">
+      <origin xyz="0.0 0.03 0.0" rpy="0 0 0"/>
+      <parent link="duo3d_left_link_${suffix}" />
+      <child link="duo3d_right_link_${suffix}" />
+      <limit upper="0" lower="0" effort="0" velocity="0" />
+      <axis xyz="0 0 1"/>
+    </joint>
+    <joint name="duo3d_optical_joint_right_${suffix}" type="revolute">
+      <origin xyz="0 0 0" rpy="${-pi/2} 0 ${-pi/2}"/>
+      <parent link="duo3d_right_link_${suffix}"/>
+      <child link="duo3d_optical_link_right_${suffix}"/>
       <limit upper="0" lower="0" effort="0" velocity="0" />
       <axis xyz="1 0 0"/>
     </joint>
-    <gazebo reference="${namespace}/duo3d_right_link">
-      <sensor name="camera" type="camera">
+    <link name="duo3d_optical_link_right_${suffix}">
+      <xacro:box_inertial x="0.0001" y="0.0001" z="0.0001" mass="0.001">
+        <origin xyz="0 0 0" rpy="0 0 0"/>
+      </xacro:box_inertial>
+      <collision>
+        <!-- todo: gazebo needs a collision volume or it will ignore the pose of
+           the joint that leads to this link (and assume it to be the identity) -->
+        <geometry>
+          <cylinder length="0.000001" radius="0.000001"/>
+        </geometry>
+        <origin xyz="0 0 0" rpy="0 ${0.5*pi} 0"/>
+      </collision>
+      <visual>
+        <geometry>
+          <cylinder length="0.000001" radius="0.000001"/>
+        </geometry>
+      </visual>
+    </link>
+    <gazebo reference="duo3d_right_link_${suffix}">
+      <sensor name="camera_${suffix}" type="camera">
       <camera>
         <horizontal_fov>${hfov}</horizontal_fov>
@@ -130,12 +193,18 @@
         </distortion>
       </camera>
-      <plugin name="right_controller" filename="libgazebo_ros_camera.so">
+      <plugin name="right_controller_${suffix}" filename="libgazebo_ros_camera.so">
         <alwaysOn>true</alwaysOn>
         <updateRate>30.0</updateRate>
-        <cameraName>${namespace}/duo3d_right</cameraName>
-        <imageTopicName>image_raw</imageTopicName>
+        <cameraName>stereo_camera_right_${suffix}</cameraName>
+        <imageTopicName>camera_image</imageTopicName>
         <cameraInfoTopicName>camera_info</cameraInfoTopicName>
-        <frameName>${namespace}/duo3d_right_link</frameName>
-        <hackBaseline>0.07</hackBaseline>
+        <frameName>/duo3d_optical_link_right_${suffix}</frameName>
+        <attenuationR>0.01</attenuationR>
+        <attenuationG>0.01</attenuationG>
+        <attenuationB>0.003</attenuationB>
+        <backgroundR>0</backgroundR>
+        <backgroundG>0</backgroundG>
+        <backgroundB>0</backgroundB>
+        <hackBaseline>0.0</hackBaseline>
         <distortionK1>${k1l}</distortionK1>
         <distortionK2>${k2l}</distortionK2>
@@ -143,4 +212,9 @@
         <distortionT1>${p1l}</distortionT1>
         <distortionT2>${p2l}</distortionT2>
+        <!-- required for ros depth cam -->
+        <pointCloudTopicName>camera_cloud</pointCloudTopicName>
+        <depthImageTopicName>camera_depth</depthImageTopicName>
+        <depthImageCameraInfoTopicName>camera_depth_info</depthImageCameraInfoTopicName>
+        <pointCloudCutoff>10.0</pointCloudCutoff>
       </plugin>
       <always_on>1</always_on>
