Commit message: Changes

File: vtec_u3_description/urdf/base.xacro (robot description, xacro)
@@ -8,17 +8,13 @@
   <xacro:include filename="$(find uuv_gazebo_ros_plugins)/urdf/snippets.xacro"/>
   <!-- Loading vehicle's specific macros -->
-  <xacro:include filename="$(find vtec_s3_description)/urdf/snippets.xacro"/>
+  <xacro:include filename="$(find vtec_u3_description)/urdf/snippets.xacro"/>
   <!--
     Vehicle's parameters (remember to enter the model parameters below)
   -->
-  <xacro:property name="mass" value="30"/>
+  <xacro:property name="mass" value="18.74"/>
   <!-- Center of gravity -->
-  <xacro:property name="cog" value="0 0 0.19"/> <!-- Superficie del barco esta a 0.19 m de COM en Z-->
+  <xacro:property name="cog" value="0 0 0"/>
   <!-- Fluid density -->
   <xacro:property name="rho" value="1000"/>
-  <!-- For the collision cube -->
-  <xacro:property name="x_size" value="1"/>
-  <xacro:property name="y_size" value="0.75"/>
-  <xacro:property name="z_size" value="0.5"/>
   <!--
     Visual mesh file for the vehicle, usually in DAE (Collada) format. Be sure to store the
@@ -27,11 +23,11 @@
     Open the meshes for the RexROV vehicle in Blender to see an example on the mesh placement.
   -->
-  <xacro:property name="visual_mesh_file" value="file://$(find vtec_s3_description)/meshes/VTECSIII_NOPROP.dae"/>
+  <xacro:property name="visual_mesh_file" value="file://$(find vtec_u3_description)/meshes/vtec_u3_spl.dae"/>
   <!-- Collision geometry mesh, usually in STL format (it is recommended to keep
   this geometry as simple as possible to improve the performance the physics engine
   regarding the computation of collision forces) -->
-  <xacro:property name="collision_mesh_file" value="file://$(find vtec_s3_description)/meshes/VTECSIII_NOPROP.stl"/>
+  <xacro:property name="collision_mesh_file" value="file://$(find vtec_u3_description)/meshes/vtec_u3_spl.stl"/>
   <!-- Vehicle macro -->
-  <xacro:macro name="vtec_s3_base" params="namespace *gazebo">
+  <xacro:macro name="vtec_u3_base" params="namespace *gazebo">
       <!-- Rigid body description of the base link -->
       <link name="${namespace}/base_link">
@@ -42,25 +38,21 @@
         <inertial>
           <mass value="${mass}" />
-          <origin xyz="0.05 0 0.19" rpy="0 0 0"/>
-          <!-- From SolidWorks -->
-          <inertia  ixx="2.5" ixy="-0.04046722475" ixz="-0.248111803"
-                    iyy="3.704654962" iyz="0.083214169"
-                    izz="4.1" />
+          <origin xyz="${cog}" rpy="0 0 0"/>
+          <inertia ixx="0.49770495" ixy="0.00275177" ixz="-0.0574426"
+                   iyy="0.37089716" iyz="-0.0036791"
+                   izz="0.64879823" />
         </inertial>
         <visual>
-          <!-- <origin xyz="0.55 -0.375 0.2" rpy="1.57075 3.141592 -1.57075"/> -->
-          <origin xyz="${cog}" rpy="0 0 0"/>
+          <origin xyz="0 0 0" rpy="0 0 0"/>
           <geometry>
-            <!-- <box size="1 0.75 0.5" />   -->
             <mesh filename="${visual_mesh_file}" scale="0.001 0.001 0.001" />
           </geometry>
         </visual>
-        <collision>
-          <origin xyz="0.05 0 0.19" rpy="0 0 0"/>
+        <!-- <collision>
+          <origin xyz="0 0 0" rpy="0 0 0"/>
           <geometry>
-            <box size="${x_size} ${y_size} ${z_size}"/>
-            <!-- <mesh filename="${collision_mesh_file}" scale="0.001 0.001 0.001" /> --> <!-- To improve performance, we replaced it by a box -->
+            <mesh filename="${collision_mesh_file}" scale="0.001 0.001 0.001" />
           </geometry>
-        </collision>
+        </collision> -->
       </link>
     <gazebo reference="${namespace}/base_link">
@@ -70,7 +62,7 @@
     <xacro:insert_block name="gazebo"/>
     <!-- Include the thruster modules -->
-    <xacro:include filename="$(find vtec_s3_description)/urdf/actuators.xacro"/>
+    <xacro:include filename="$(find vtec_u3_description)/urdf/actuators.xacro"/>
     <!-- Include the sensor modules -->
-    <!-- <xacro:include filename="$(find vtec_s3_description)/urdf/sensors.xacro"/> -->
+    <xacro:include filename="$(find vtec_u3_description)/urdf/sensors.xacro"/>
   </xacro:macro>
 </robot>
